File: Divider.kicad_pcb (KiCad board)
At the start: 2 copper layers, 73 parts, among them J1 AudioJack2_SwitchT, J10 AudioJack2_SwitchT, J11 Conn_02x03_Odd_Even, J12 Conn_02x05_Odd_Even, J2 AudioJack2_SwitchT, J3 AudioJack2_SwitchT, J4 AudioJack2_SwitchT, J5 AudioJack2_SwitchT, J6 AudioJack2_SwitchT, J7 AudioJack2_SwitchT, J8 AudioJack2_SwitchT, J9 AudioJack2_SwitchT, Q1 BC847, Q2 BC847, SW1 SW_Push, SW2 SW_SPDT_MSM, SW3 SW_SPDT_MSM, U1 ATtiny84-20MU, U10 74AHCT1G125, U2 74AHCT1G125, U3 L7805, U4 74AHCT1G125, U5 74AHCT1G125, U6 74AHCT1G125, U7 74AHCT1G125, U8 74AHCT1G125, U9 74AHCT1G125

Commit message: Initial placement.
Parts:
- removed C6: 10u, Capacitor_SMD:CP_Elec_4x5.8
- removed D5: DFLR1400-7, Diode_SMD:D_PowerDI-123
- C1, C2, C3, C4, C5, C7, D3, D4, J11, J12, Q1, Q2, R1, R10, R11, R12, R13, R14, R15, R16, R17, R18, R19, R20, R21, R22, R23, R24, R25, R26, R27, R28, R29, R3, R4, R5, R6, R7, R8, R9, U1, U10, U2, U3, U4, U5, U6, U7, U8, U9: moved to B.Cu
- moved U8 157.5 mm to (137.7, 145.8), turned to 180 degrees
- moved R24 156.5 mm to (133.8, 149.4)
- moved R25 154.9 mm to (141.4, 149.4)
- moved U9 149.5 mm to (158.2, 132.2), turned to 180 degrees
- moved R26 148.6 mm to (154.2, 135.9)
- moved U4 147.2 mm to (137.6, 118.5), turned to 180 degrees
- moved R27 147.1 mm to (161.7, 135.9)
- moved R14 146.3 mm to (133.8, 88.1), turned to 180 degrees
- moved R16 146.1 mm to (133.8, 122.3)
- moved D10 144.9 mm to (143.5, 140.6)
- moved R28 144.4 mm to (133.8, 135.9)
- moved R17 144.3 mm to (141.4, 122.3)
- moved R15 143.7 mm to (133.9, 79.6), turned to 180 degrees
- moved U10 140.8 mm to (137.7, 132.2), turned to 180 degrees
- moved R7 138.7 mm to (141.1, 58.8), turned to 90 degrees
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Connections:
- C1 pad 2: GND -> (no net)
- C2 pad 2: GND -> (no net)
- C3 pad 2: GND -> (no net)
- C4 pad 2: GND -> (no net)
- C5 pad 2: GND -> (no net)
- C7 pad 2: GND -> (no net)
- D10 pad 1: GND -> (no net)
- D11 pad 1: GND -> (no net)
- D12 pad 1: GND -> (no net)
- D2 pad 1: GND -> (no net)
- D4 pad 1: GND -> (no net)
- D6 pad 1: GND -> (no net)
- D7 pad 1: GND -> (no net)
- D8 pad 1: GND -> (no net)
- D9 pad 1: GND -> (no net)
- J1 pad S: GND -> (no net)
- J10 pad S: GND -> (no net)
- J11 pad 6: GND -> (no net)
- J12 pad 3: GND -> (no net)
- J12 pad 4: GND -> (no net)
- J12 pad 5: GND -> (no net)
- J12 pad 6: GND -> (no net)
- J12 pad 7: GND -> (no net)
- J12 pad 8: GND -> (no net)
- J2 pad S: GND -> (no net)
- J3 pad S: GND -> (no net)
- J4 pad S: GND -> (no net)
- J5 pad S: GND -> (no net)
- J6 pad S: GND -> (no net)
- J7 pad S: GND -> (no net)
- J7 pad TN: GND -> (no net)
- J8 pad S: GND -> (no net)
- J9 pad S: GND -> (no net)
- Q1 pad 2: GND -> (no net)
- Q2 pad 2: GND -> (no net)
- R12 pad 2: GND -> (no net)
- R13 pad 2: GND -> (no net)
- SW1 pad 2: GND -> (no net)
- U1 pad 21: GND -> (no net)
- U1 pad 8: GND -> (no net)
- U10 pad 1: GND -> (no net)
- U10 pad 3: GND -> (no net)
- U2 pad 1: GND -> (no net)
- U2 pad 3: GND -> (no net)
- U3 pad 2: GND -> (no net)
- U4 pad 1: GND -> (no net)
- U4 pad 3: GND -> (no net)
- U5 pad 1: GND -> (no net)
- U5 pad 3: GND -> (no net)
- U6 pad 1: GND -> (no net)
- U6 pad 3: GND -> (no net)
- U7 pad 1: GND -> (no net)
- U7 pad 3: GND -> (no net)
- U8 pad 1: GND -> (no net)
- U8 pad 3: GND -> (no net)
- U9 pad 1: GND -> (no net)
- U9 pad 3: GND -> (no net)
Other:
- board outline added: 39.6 x 100 mm

Commit message: Manual power routing.
Parts:
- moved SW1 7.91 mm to (151.8, 76.8), turned to 180 degrees
- turned D3 to 270 degrees
- turned R3 to 180 degrees
Connections:
- U1 pad 11: OUT7 -> OUT2
- U1 pad 14: RST -> OUT0
- U1 pad 2: OUT3 -> RST
- U1 pad 3: OUT2 -> OUT1
- U1 pad 4: OUT1 -> OUT3
- U1 pad 5: OUT0 -> OUT7
Routing:
- net +5V: track 0.00 -> 61.2 mm
- net +12V: track 0.00 -> 52.1 mm
- net Net-(D3-Pad2): track 0.00 -> 6.92 mm
- net Net-(J12-Pad1): track 0.00 -> 2.54 mm

Commit message: Complete signal routing.
Parts:
- moved R1 9.02 mm to (133.9, 88.1)
- moved R14 2.80 mm to (133.9, 85.3)
Routing:
- net +5V: track 61.2 -> 266.4 mm
- net MOSI: track 0.00 -> 85.7 mm, vias 0 -> 1
- net MISO: track 0.00 -> 82.1 mm
- net OUT7: track 0.00 -> 77.8 mm, vias 0 -> 2
- net OUT4: track 0.00 -> 75.3 mm
- net RESET: track 0.00 -> 65.2 mm, vias 0 -> 2
- net SPDTS: track 0.00 -> 53.6 mm, vias 0 -> 4
- net Net-(R10-Pad1): track 0.00 -> 37.8 mm, vias 0 -> 1
- net CLK: track 0.00 -> 32.9 mm, vias 0 -> 2
- net OUT2: track 0.00 -> 30.9 mm
- net OUT3: track 0.00 -> 29.4 mm, vias 0 -> 2
- net OUT0: track 0.00 -> 27.4 mm
- net RST: track 0.00 -> 18.9 mm
- net OUT1: track 0.00 -> 17.6 mm, vias 0 -> 2
- net Net-(D11-Pad2): track 0.00 -> 12.0 mm
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
Commit message: Ground pours.
Connections:
- C1 pad 2: (no net) -> GND
- C2 pad 2: (no net) -> GND
- C3 pad 2: (no net) -> GND
- C4 pad 2: (no net) -> GND
- C5 pad 2: (no net) -> GND
- C7 pad 2: (no net) -> GND
- D10 pad 1: (no net) -> GND
- D11 pad 1: (no net) -> GND
- D12 pad 1: (no net) -> GND
- D2 pad 1: (no net) -> GND
- D4 pad 1: (no net) -> GND
- D6 pad 1: (no net) -> GND
- D7 pad 1: (no net) -> GND
- D8 pad 1: (no net) -> GND
- D9 pad 1: (no net) -> GND
- J1 pad S: (no net) -> GND
- J10 pad S: (no net) -> GND
- J11 pad 6: (no net) -> GND
- J12 pad 3: (no net) -> GND
- J12 pad 4: (no net) -> GND
- J12 pad 5: (no net) -> GND
- J12 pad 6: (no net) -> GND
- J12 pad 7: (no net) -> GND
- J12 pad 8: (no net) -> GND
- J2 pad S: (no net) -> GND
- J3 pad S: (no net) -> GND
- J4 pad S: (no net) -> GND
- J5 pad S: (no net) -> GND
- J6 pad S: (no net) -> GND
- J7 pad S: (no net) -> GND
- J7 pad TN: (no net) -> GND
- J8 pad S: (no net) -> GND
- J9 pad S: (no net) -> GND
- Q1 pad 2: (no net) -> GND
- Q2 pad 2: (no net) -> GND
- R12 pad 2: (no net) -> GND
- R13 pad 2: (no net) -> GND
- SW1 pad 2: (no net) -> GND
- U1 pad 21: (no net) -> GND
- U1 pad 8: (no net) -> GND
- U10 pad 1: (no net) -> GND
- U10 pad 3: (no net) -> GND
- U2 pad 1: (no net) -> GND
- U2 pad 3: (no net) -> GND
- U3 pad 2: (no net) -> GND
- U4 pad 1: (no net) -> GND
- U4 pad 3: (no net) -> GND
- U5 pad 1: (no net) -> GND
- U5 pad 3: (no net) -> GND
- U6 pad 1: (no net) -> GND
- U6 pad 3: (no net) -> GND
- U7 pad 1: (no net) -> GND
- U7 pad 3: (no net) -> GND
- U8 pad 1: (no net) -> GND
- U8 pad 3: (no net) -> GND
- U9 pad 1: (no net) -> GND
- U9 pad 3: (no net) -> GND
Routing:
- net GND: track 0.00 -> 32.5 mm, vias 0 -> 25
- net RESET: track 65.2 -> 68.9 mm
- net +5V: track 266.4 -> 264.1 mm
- net Net-(R10-Pad1): track 37.8 -> 35.6 mm
- net RST: track 18.9 -> 19.4 mm
- added copper zone on B.Cu, net GND
- added copper zone on F.Cu, net GND

Commit message: Improved pour.
Routing:
- net MISO: track 82.2 -> 82.9 mm
- net GND: vias 25 -> 26
Changed lines of the file:
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@@
     (thickness 1.6)
     (drawings 70)
-    (tracks 545)
+    (tracks 557)
     (zones 0)
     (modules 71)
@@
   (segment (start 134.911 96.11) (end 136.689 96.11) (width 0.25) (layer B.Cu) (net 12))
   (segment (start 136.689 96.11) (end 138.895 93.904) (width 0.25) (layer B.Cu) (net 12))
-  (segment (start 138.805 145.767) (end 138.025 145.767) (width 0.25) (layer B.Cu) (net 12))
-  (segment (start 138.025 145.767) (end 135.8 145.767) (width 0.25) (layer B.Cu) (net 12))
-  (segment (start 135.8 145.767) (end 134.911 144.878) (width 0.25) (layer B.Cu) (net 12))
-  (segment (start 134.911 144.878) (end 134.911 141.068) (width 0.25) (layer B.Cu) (net 12))
-  (segment (start 134.911 141.068) (end 129.577 135.734) (width 0.25) (layer B.Cu) (net 12))
   (via (at 130.212 94.967) (size 0.8) (drill 0.4) (layers F.Cu B.Cu) (net 12))
-  (segment (start 129.577 135.734) (end 129.577 95.602) (width 0.25) (layer B.Cu) (net 12))
-  (segment (start 129.577 95.602) (end 130.212 94.967) (width 0.25) (layer B.Cu) (net 12))
   (segment (start 140.245 149.0945) (end 140.6005 149.45) (width 0.25) (layer B.Cu) (net 12))
   (segment (start 138.805 145.767) (end 139.737 145.767) (width 0.25) (layer B.Cu) (net 12))
@@
   (segment (start 130.212 94.967) (end 130.777685 94.967) (width 0.25) (layer F.Cu) (net 12))
   (segment (start 130.777685 94.967) (end 130.904685 94.84) (width 0.25) (layer F.Cu) (net 12))
+  (segment (start 130.085 95.094) (end 130.212 94.967) (width 0.25) (layer B.Cu) (net 12))
+  (segment (start 131.355 102.841) (end 130.085 101.571) (width 0.25) (layer B.Cu) (net 12))
+  (segment (start 130.085 101.571) (end 130.085 95.094) (width 0.25) (layer B.Cu) (net 12))
+  (segment (start 131.355 112.112) (end 131.355 102.841) (width 0.25) (layer B.Cu) (net 12))
+  (segment (start 135.8 145.767) (end 135.165 145.132) (width 0.25) (layer B.Cu) (net 12))
+  (segment (start 131.99 138.147) (end 131.99 112.747) (width 0.25) (layer B.Cu) (net 12))
+  (segment (start 131.99 112.747) (end 131.355 112.112) (width 0.25) (layer B.Cu) (net 12))
+  (segment (start 138.805 145.767) (end 135.8 145.767) (width 0.25) (layer B.Cu) (net 12))
+  (segment (start 135.165 145.132) (end 135.165 141.322) (width 0.25) (layer B.Cu) (net 12))
+  (segment (start 135.165 141.322) (end 131.99 138.147) (width 0.25) (layer B.Cu) (net 12))
   (segment (start 153.74 132.051) (end 153.74 133.6763) (width 0.25) (layer B.Cu) (net 13))
   (segment (start 153.74 133.6763) (end 153.4275 133.9888) (width 0.25) (layer B.Cu) (net 13))
@@
   (segment (start 159.252 132.178) (end 160.057 132.178) (width 0.25) (layer B.Cu) (net 16))
   (segment (start 160.057 132.178) (end 160.819 132.94) (width 0.25) (layer B.Cu) (net 16))
-  (segment (start 148.8878 124.4068) (end 156.659 132.178) (width 0.25) (layer B.Cu) (net 16))
+  (segment (start 133.91999 111.88299) (end 135.413 113.376) (width 0.25) (layer B.Cu) (net 16))
+  (segment (start 133.91999 107.51501) (end 133.91999 111.88299) (width 0.25) (layer B.Cu) (net 16))
+  (segment (start 134.784 106.651) (end 133.91999 107.51501) (width 0.25) (layer B.Cu) (net 16))
+  (segment (start 134.784 102.163) (end 134.784 106.651) (width 0.25) (layer B.Cu) (net 16))
+  (segment (start 137.333001 118.826999) (end 137.333001 119.997001) (width 0.25) (layer B.Cu) (net 16))
+  (segment (start 132.371 99.75) (end 134.784 102.163) (width 0.25) (layer B.Cu) (net 16))
+  (segment (start 136.048 118.462) (end 136.968002 118.462) (width 0.25) (layer B.Cu) (net 16))
+  (segment (start 132.371 98.65) (end 132.371 99.75) (width 0.25) (layer B.Cu) (net 16))
+  (segment (start 135.413 113.376) (end 135.413 117.827) (width 0.25) (layer B.Cu) (net 16))
+  (segment (start 135.413 117.827) (end 136.048 118.462) (width 0.25) (layer B.Cu) (net 16))
+  (segment (start 137.324 120.006002) (end 137.324 120.2647) (width 0.25) (layer B.Cu) (net 16))
   (segment (start 141.4661 124.4068) (end 148.8878 124.4068) (width 0.25) (layer B.Cu) (net 16))
+  (segment (start 136.968002 118.462) (end 137.333001 118.826999) (width 0.25) (layer B.Cu) (net 16))
   (segment (start 137.333001 119.997001) (end 137.324 120.006002) (width 0.25) (layer B.Cu) (net 16))
-  (segment (start 132.371 99.8253) (end 132.2914 99.9049) (width 0.25) (layer B.Cu) (net 16))
   (segment (start 137.324 120.2647) (end 141.4661 124.4068) (width 0.25) (layer B.Cu) (net 16))
-  (segment (start 137.324 120.006002) (end 137.324 120.2647) (width 0.25) (layer B.Cu) (net 16))
-  (segment (start 136.048 118.462) (end 136.968002 118.462) (width 0.25) (layer B.Cu) (net 16))
   (segment (start 156.659 132.178) (end 159.252 132.178) (width 0.25) (layer B.Cu) (net 16))
-  (segment (start 137.333001 118.826999) (end 137.333001 119.997001) (width 0.25) (layer B.Cu) (net 16))
-  (segment (start 132.371 98.65) (end 132.371 99.8253) (width 0.25) (layer B.Cu) (net 16))
-  (segment (start 132.2914 99.9049) (end 132.2914 114.7054) (width 0.25) (layer B.Cu) (net 16))
-  (segment (start 132.2914 114.7054) (end 136.048 118.462) (width 0.25) (layer B.Cu) (net 16))
-  (segment (start 136.968002 118.462) (end 137.333001 118.826999) (width 0.25) (layer B.Cu) (net 16))
+  (segment (start 148.8878 124.4068) (end 156.659 132.178) (width 0.25) (layer B.Cu) (net 16))
   (segment (start 133.42 132.051) (end 133.42 133.6763) (width 0.25) (layer B.Cu) (net 17))
   (segment (start 133.42 133.6763) (end 132.9805 134.1158) (width 0.25) (layer B.Cu) (net 17))
@@
   (segment (start 134.276 91.792) (end 133.641 92.427) (width 0.25) (layer B.Cu) (net 20))
   (segment (start 140.118 131.6077) (end 139.5477 132.178) (width 0.25) (layer B.Cu) (net 20))
-  (segment (start 140.118 130.273) (end 140.118 131.6077) (width 0.25) (layer B.Cu) (net 20))
+  (segment (start 133.79299 121.790516) (end 133.79299 123.94799) (width 0.25) (layer B.Cu) (net 20))
   (segment (start 131.736 96.11) (end 130.72 97.126) (width 0.25) (layer B.Cu) (net 20))
+  (segment (start 134.784 120.799506) (end 133.79299 121.790516) (width 0.25) (layer B.Cu) (net 20))
+  (segment (start 130.72 101.063) (end 131.99 102.333) (width 0.25) (layer B.Cu) (net 20))
+  (segment (start 140.118 130.273) (end 140.118 131.6077) (width 0.25) (layer B.Cu) (net 20))
+  (segment (start 133.79299 123.94799) (end 140.118 130.273) (width 0.25) (layer B.Cu) (net 20))
   (segment (start 132.371 96.11) (end 131.736 96.11) (width 0.25) (layer B.Cu) (net 20))
-  (segment (start 130.72 97.126) (end 130.72 122.272) (width 0.25) (layer B.Cu) (net 20))
-  (segment (start 130.72 122.272) (end 131.99 123.542) (width 0.25) (layer B.Cu) (net 20))
-  (segment (start 133.387 123.542) (end 140.118 130.273) (width 0.25) (layer B.Cu) (net 20))
-  (segment (start 131.99 123.542) (end 133.387 123.542) (width 0.25) (layer B.Cu) (net 20))
+  (segment (start 134.784 114.271) (end 134.784 120.799506) (width 0.25) (layer B.Cu) (net 20))
+  (segment (start 130.72 97.126) (end 130.72 101.063) (width 0.25) (layer B.Cu) (net 20))
+  (segment (start 131.99 102.333) (end 131.99 111.477) (width 0.25) (layer B.Cu) (net 20))
+  (segment (start 131.99 111.477) (end 134.784 114.271) (width 0.25) (layer B.Cu) (net 20))
   (segment (start 138.551 105) (end 139.4063 105) (width 0.25) (layer B.Cu) (net 21))
   (segment (start 140.118 108.3275) (end 140.6005 108.81) (width 0.25) (layer B.Cu) (net 21))
@@
   (via (at 160.565 130.273) (size 0.8) (drill 0.4) (layers F.Cu B.Cu) (net 63))
   (via (at 164.375 60.042) (size 0.8) (drill 0.4) (layers F.Cu B.Cu) (net 63))
+  (via (at 130.847 75.028) (size 0.8) (drill 0.4) (layers F.Cu B.Cu) (net 63))
   (zone (net 63) (net_name GND) (layer F.Cu) (hatch edge 0.508)
     (connect_pads (clearance 0.508))
