File: Divider.kicad_pcb (KiCad board)
At the start: 2 copper layers, 39.6 x 100 mm, 71 parts, among them J1 AudioJack2_SwitchT, J10 AudioJack2_SwitchT, J11 Conn_02x03_Odd_Even, J12 Conn_02x05_Odd_Even, J2 AudioJack2_SwitchT, J3 AudioJack2_SwitchT, J4 AudioJack2_SwitchT, J5 AudioJack2_SwitchT, J6 AudioJack2_SwitchT, J7 AudioJack2_SwitchT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

Commit message: Branding.
Other:
- board text added: "-12V"
- board text added: "Divider"
- board text added: "ICSP"
- board text added: "Marangisto 2019"
- board text added: "Rev A"
Changed lines of the file:
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@@
   (general
     (thickness 1.6)
-    (drawings 70)
+    (drawings 76)
     (tracks 557)
     (zones 0)
@@
     )
   )
+  (gr_text ICSP (at 137.578 96.11 90) (layer B.SilkS)
+    (effects (font (size 1 1) (thickness 0.2)) (justify mirror))
+  )
+  (gr_text -12V (at 143.42 69.186) (layer B.SilkS)
+    (effects (font (size 1 1) (thickness 0.2)) (justify mirror))
+  )
+  (gr_line (start 150.786 70.964) (end 146.214 70.964) (layer B.SilkS) (width 0.4))
+  (gr_text "Rev A" (at 166.28 151.482 90) (layer B.SilkS)
+    (effects (font (size 1 1) (thickness 0.2)) (justify mirror))
+  )
+  (gr_text "Marangisto 2019" (at 166.28 62.836 90) (layer B.SilkS)
+    (effects (font (size 1 1) (thickness 0.2)) (justify mirror))
+  )
+  (gr_text Divider (at 130.72 74.774 90) (layer B.SilkS)
+    (effects (font (size 2 6) (thickness 0.3)) (justify mirror))
+  )
   (target plus (at 148.5 105) (size 5) (width 0.15) (layer Edge.Cuts))
   (target plus (at 148.5 105) (size 5) (width 0.15) (layer Edge.Cuts))
@@
   (gr_line (start 128.6811 55.0036) (end 128.6811 155.0036) (layer Edge.Cuts) (width 0.2))
   (gr_line (start 168.3211 155.0036) (end 168.3211 55.0036) (layer Edge.Cuts) (width 0.2))
-  (via (at 150.405 89.887) (size 0.8) (drill 0.4) (layers F.Cu B.Cu) (net 63))
-  (via (at 148.373 89.887) (size 0.8) (drill 0.4) (layers F.Cu B.Cu) (net 63))
-  (via (at 146.595 89.887) (size 0.8) (drill 0.4) (layers F.Cu B.Cu) (net 63))
-  (via (at 150.405 87.855) (size 0.8) (drill 0.4) (layers F.Cu B.Cu) (net 63))
-  (via (at 148.373 87.855) (size 0.8) (drill 0.4) (layers F.Cu B.Cu) (net 63))
-  (via (at 146.595 87.855) (size 0.8) (drill 0.4) (layers F.Cu B.Cu) (net 63))
-  (via (at 150.151 85.823) (size 0.8) (drill 0.4) (layers F.Cu B.Cu) (net 63))
-  (via (at 148.373 85.823) (size 0.8) (drill 0.4) (layers F.Cu B.Cu) (net 63))
-  (via (at 146.595 85.823) (size 0.8) (drill 0.4) (layers F.Cu B.Cu) (net 63))
-  (via (at 152.818 97.126) (size 0.8) (drill 0.4) (layers F.Cu B.Cu) (net 63))
-  (via (at 153.834 97.126) (size 0.8) (drill 0.4) (layers F.Cu B.Cu) (net 63))
-  (via (at 153.834 96.11) (size 0.8) (drill 0.4) (layers F.Cu B.Cu) (net 63))
-  (via (at 152.818 96.11) (size 0.8) (drill 0.4) (layers F.Cu B.Cu) (net 63))
   (segment (start 157.308 96.618) (end 155.2635 96.618) (width 0.25) (layer B.Cu) (net 1))
   (via (at 158.406 96.618) (size 0.8) (drill 0.4) (layers F.Cu B.Cu) (net 1))
@@
   (segment (start 149.795 58.772) (end 147.255 58.772) (width 1) (layer B.Cu) (net 61))
   (segment (start 149.795 68.932) (end 147.255 68.932) (width 1) (layer B.Cu) (net 62))
+  (via (at 150.405 89.887) (size 0.8) (drill 0.4) (layers F.Cu B.Cu) (net 63))
+  (via (at 148.373 89.887) (size 0.8) (drill 0.4) (layers F.Cu B.Cu) (net 63))
+  (via (at 146.595 89.887) (size 0.8) (drill 0.4) (layers F.Cu B.Cu) (net 63))
+  (via (at 150.405 87.855) (size 0.8) (drill 0.4) (layers F.Cu B.Cu) (net 63))
+  (via (at 148.373 87.855) (size 0.8) (drill 0.4) (layers F.Cu B.Cu) (net 63))
+  (via (at 146.595 87.855) (size 0.8) (drill 0.4) (layers F.Cu B.Cu) (net 63))
+  (via (at 150.151 85.823) (size 0.8) (drill 0.4) (layers F.Cu B.Cu) (net 63))
+  (via (at 148.373 85.823) (size 0.8) (drill 0.4) (layers F.Cu B.Cu) (net 63))
+  (via (at 146.595 85.823) (size 0.8) (drill 0.4) (layers F.Cu B.Cu) (net 63))
+  (via (at 152.818 97.126) (size 0.8) (drill 0.4) (layers F.Cu B.Cu) (net 63))
+  (via (at 153.834 97.126) (size 0.8) (drill 0.4) (layers F.Cu B.Cu) (net 63))
+  (via (at 153.834 96.11) (size 0.8) (drill 0.4) (layers F.Cu B.Cu) (net 63))
+  (via (at 152.818 96.11) (size 0.8) (drill 0.4) (layers F.Cu B.Cu) (net 63))
   (segment (start 153.326 98.5555) (end 153.326 96.618) (width 0.25) (layer B.Cu) (net 63))
   (via (at 151.294 102.46) (size 0.8) (drill 0.4) (layers F.Cu B.Cu) (net 63))
